File: device/POC/BikeLight POC.sch (EAGLE design)
At the start: 43 parts, among them IC1 MCP2515-I-ML, IC10 MCP1802T-5002I/OT, IC2 MICROSD_SPI_MODE, IC3 FM25W256-SOIC, IC4 MCP2561-2, IC5 TXB0106, IC6 PRQV8.00CR1510Y00L, IC7 ADXL345, IC8 74HCT1G32, IC9 MCP1802T-3302I/OT

Commit message: - finished layout (silk top and bottom) - created gerbers
Parts:
- removed TP5, TP6, TP7, TP9: TPPAD1-13, testpad:TPPAD1-13
- added CAN_GND, MISO, MOSI, SCK: PTR1PAD1-13Y, testpad:PTR1PAD1-13Y
- TP1, TP2, TP3, TP4: value PTR1PAD1-13Y -> TPPAD1-13; device testpad:PTR1PAD1-13Y -> testpad:TPPAD1-13
- renumbered S1 to POWER
Connections:
- net GND: now also CAN_GND.TP; no longer TP1.TP
- net P0.15-SPI_MISO: now also MISO.TP; no longer TP3.TP
- net P0.16-SPI_MOSI: now also MOSI.TP; no longer TP2.TP
- net P0.17-SPI_SCK: now also SCK.TP; no longer TP4.TP
- net P0.18-SPI_SS_MCP2515: now also TP4.TP; no longer TP7.TP
- net P0.23-SPI_SS_ADXL345_PIN: now also TP3.TP; no longer TP5.TP
- net P0.24-SPI_SS_FRAM: now also TP2.TP; no longer TP6.TP
- net P0.25-SPI_SS_SD-CARD: now also TP1.TP; no longer TP9.TP
Changed lines of the file:
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@@
 <part name="C10" library="rcl" library_urn="urn:adsk.eagle:library:334" deviceset="C-EU" device="C0805" package3d_urn="urn:adsk.eagle:package:23617/2" value="4.7μF"/>
 <part name="C11" library="rcl" library_urn="urn:adsk.eagle:library:334" deviceset="C-EU" device="C0805" package3d_urn="urn:adsk.eagle:package:23617/2" value="4.7μF"/>
-<part name="S1" library="smd-special" library_urn="urn:adsk.eagle:library:362" deviceset="SWS001" device="" package3d_urn="urn:adsk.eagle:package:26467/1"/>
+<part name="POWER" library="smd-special" library_urn="urn:adsk.eagle:library:362" deviceset="SWS001" device="" package3d_urn="urn:adsk.eagle:package:26467/1"/>
 <part name="R8" library="rcl" library_urn="urn:adsk.eagle:library:334" deviceset="R-EU_" device="R0805" package3d_urn="urn:adsk.eagle:package:23553/2" value="100k"/>
 <part name="IC8" library="74HCT1G32GW - OR Gate" deviceset="74HCT1G32GW" device="-DC" value="74HCT1G32"/>
-<part name="TP1" library="testpad" library_urn="urn:adsk.eagle:library:385" deviceset="PTR1" device="PAD1-13Y" package3d_urn="urn:adsk.eagle:package:27947/1"/>
-<part name="TP2" library="testpad" library_urn="urn:adsk.eagle:library:385" deviceset="PTR1" device="PAD1-13Y" package3d_urn="urn:adsk.eagle:package:27947/1"/>
-<part name="TP3" library="testpad" library_urn="urn:adsk.eagle:library:385" deviceset="PTR1" device="PAD1-13Y" package3d_urn="urn:adsk.eagle:package:27947/1"/>
-<part name="TP4" library="testpad" library_urn="urn:adsk.eagle:library:385" deviceset="PTR1" device="PAD1-13Y" package3d_urn="urn:adsk.eagle:package:27947/1"/>
-<part name="TP5" library="testpad" library_urn="urn:adsk.eagle:library:385" deviceset="TP" device="PAD1-13" package3d_urn="urn:adsk.eagle:package:27946/1"/>
-<part name="TP6" library="testpad" library_urn="urn:adsk.eagle:library:385" deviceset="TP" device="PAD1-13" package3d_urn="urn:adsk.eagle:package:27946/1"/>
-<part name="TP7" library="testpad" library_urn="urn:adsk.eagle:library:385" deviceset="TP" device="PAD1-13" package3d_urn="urn:adsk.eagle:package:27946/1"/>
-<part name="TP9" library="testpad" library_urn="urn:adsk.eagle:library:385" deviceset="TP" device="PAD1-13" package3d_urn="urn:adsk.eagle:package:27946/1"/>
+<part name="CAN_GND" library="testpad" library_urn="urn:adsk.eagle:library:385" deviceset="PTR1" device="PAD1-13Y" package3d_urn="urn:adsk.eagle:package:27947/1"/>
+<part name="MOSI" library="testpad" library_urn="urn:adsk.eagle:library:385" deviceset="PTR1" device="PAD1-13Y" package3d_urn="urn:adsk.eagle:package:27947/1" value=""/>
+<part name="MISO" library="testpad" library_urn="urn:adsk.eagle:library:385" deviceset="PTR1" device="PAD1-13Y" package3d_urn="urn:adsk.eagle:package:27947/1" value=""/>
+<part name="SCK" library="testpad" library_urn="urn:adsk.eagle:library:385" deviceset="PTR1" device="PAD1-13Y" package3d_urn="urn:adsk.eagle:package:27947/1" value=""/>
+<part name="TP3" library="testpad" library_urn="urn:adsk.eagle:library:385" deviceset="TP" device="PAD1-13" package3d_urn="urn:adsk.eagle:package:27946/1" value=""/>
+<part name="TP2" library="testpad" library_urn="urn:adsk.eagle:library:385" deviceset="TP" device="PAD1-13" package3d_urn="urn:adsk.eagle:package:27946/1" value=""/>
+<part name="TP4" library="testpad" library_urn="urn:adsk.eagle:library:385" deviceset="TP" device="PAD1-13" package3d_urn="urn:adsk.eagle:package:27946/1" value=""/>
+<part name="TP1" library="testpad" library_urn="urn:adsk.eagle:library:385" deviceset="TP" device="PAD1-13" package3d_urn="urn:adsk.eagle:package:27946/1" value=""/>
 <part name="LED1" library="led" library_urn="urn:adsk.eagle:library:259" deviceset="LED" device="CHIPLED_1206" package3d_urn="urn:adsk.eagle:package:15823/2" value="  LTST-C230KSKT"/>
 <part name="R9" library="rcl" library_urn="urn:adsk.eagle:library:334" deviceset="R-EU_" device="R0805" package3d_urn="urn:adsk.eagle:package:23553/2" value="10k"/>
@@
 <instance part="C10" gate="G$1" x="81.28" y="-101.6" rot="R180"/>
 <instance part="C11" gate="G$1" x="119.38" y="-101.6" rot="R180"/>
-<instance part="S1" gate="G$1" x="93.98" y="-170.18" rot="R90"/>
+<instance part="POWER" gate="G$1" x="93.98" y="-170.18" rot="R90"/>
 <instance part="R8" gate="G$1" x="101.6" y="-175.26" rot="R90"/>
 <instance part="IC8" gate="G$1" x="365.76" y="-48.26" rot="R180"/>
-<instance part="TP1" gate="G$1" x="-7.62" y="-68.58" rot="R270"/>
-<instance part="TP2" gate="G$1" x="-7.62" y="-78.74" rot="R270"/>
-<instance part="TP3" gate="G$1" x="-7.62" y="-88.9" rot="R270"/>
-<instance part="TP4" gate="G$1" x="-7.62" y="-99.06" rot="R270"/>
-<instance part="TP5" gate="G$1" x="-7.62" y="-109.22" rot="R270"/>
-<instance part="TP6" gate="G$1" x="-7.62" y="-119.38" rot="R270"/>
-<instance part="TP7" gate="G$1" x="-7.62" y="-129.54" rot="R270"/>
-<instance part="TP9" gate="G$1" x="-7.62" y="-139.7" rot="R270"/>
+<instance part="CAN_GND" gate="G$1" x="-7.62" y="-68.58" rot="R270"/>
+<instance part="MOSI" gate="G$1" x="-7.62" y="-78.74" rot="R270"/>
+<instance part="MISO" gate="G$1" x="-7.62" y="-88.9" rot="R270"/>
+<instance part="SCK" gate="G$1" x="-7.62" y="-99.06" rot="R270"/>
+<instance part="TP3" gate="G$1" x="-7.62" y="-124.46" rot="R90"/>
+<instance part="TP2" gate="G$1" x="-7.62" y="-116.84" rot="R90"/>
+<instance part="TP4" gate="G$1" x="-7.62" y="-132.08" rot="R90"/>
+<instance part="TP1" gate="G$1" x="-7.62" y="-109.22" rot="R90"/>
 <instance part="LED1" gate="G$1" x="101.6" y="-165.1" rot="R180"/>
 <instance part="R9" gate="G$1" x="101.6" y="-154.94" rot="R90"/>
@@
 </segment>
 <segment>
-<pinref part="TP1" gate="G$1" pin="TP"/>
+<pinref part="CAN_GND" gate="G$1" pin="TP"/>
 <wire x1="-5.08" y1="-68.58" x2="0" y2="-68.58" width="0.1524" layer="91"/>
 <label x="0" y="-68.58" size="1.778" layer="95"/>
@@
 </segment>
 <segment>
-<pinref part="S1" gate="G$1" pin="2"/>
+<pinref part="POWER" gate="G$1" pin="2"/>
 <wire x1="86.36" y1="-170.18" x2="68.58" y2="-170.18" width="0.1524" layer="91"/>
 <label x="68.58" y="-170.18" size="1.778" layer="95"/>
@@
 </segment>
 <segment>
-<pinref part="TP6" gate="G$1" pin="TP"/>
-<wire x1="-10.16" y1="-119.38" x2="0" y2="-119.38" width="0.1524" layer="91"/>
-<label x="0" y="-119.38" size="1.778" layer="95"/>
+<pinref part="TP2" gate="G$1" pin="TP"/>
+<wire x1="-5.08" y1="-116.84" x2="0" y2="-116.84" width="0.1524" layer="91"/>
+<label x="0" y="-116.84" size="1.778" layer="95"/>
 </segment>
 </net>
@@
 </segment>
 <segment>
-<pinref part="S1" gate="G$1" pin="1"/>
+<pinref part="POWER" gate="G$1" pin="1"/>
 <wire x1="99.06" y1="-170.18" x2="101.6" y2="-170.18" width="0.1524" layer="91"/>
 <label x="109.22" y="-170.18" size="1.778" layer="95"/>
@@
 </segment>
 <segment>
-<pinref part="TP7" gate="G$1" pin="TP"/>
-<wire x1="-10.16" y1="-129.54" x2="0" y2="-129.54" width="0.1524" layer="91"/>
-<label x="0" y="-129.54" size="1.778" layer="95"/>
+<pinref part="TP4" gate="G$1" pin="TP"/>
+<wire x1="-5.08" y1="-132.08" x2="0" y2="-132.08" width="0.1524" layer="91"/>
+<label x="0" y="-132.08" size="1.778" layer="95"/>
 </segment>
 </net>
@@
 </segment>
 <segment>
-<pinref part="TP4" gate="G$1" pin="TP"/>
+<pinref part="SCK" gate="G$1" pin="TP"/>
 <wire x1="-5.08" y1="-99.06" x2="0" y2="-99.06" width="0.1524" layer="91"/>
 <label x="0" y="-99.06" size="1.778" layer="95"/>
@@
 </segment>
 <segment>
-<pinref part="TP9" gate="G$1" pin="TP"/>
-<wire x1="-10.16" y1="-139.7" x2="0" y2="-139.7" width="0.1524" layer="91"/>
-<label x="0" y="-139.7" size="1.778" layer="95"/>
+<pinref part="TP1" gate="G$1" pin="TP"/>
+<wire x1="-5.08" y1="-109.22" x2="0" y2="-109.22" width="0.1524" layer="91"/>
+<label x="0" y="-109.22" size="1.778" layer="95"/>
 </segment>
 </net>
@@
 </segment>
 <segment>
-<pinref part="TP5" gate="G$1" pin="TP"/>
-<wire x1="-10.16" y1="-109.22" x2="0" y2="-109.22" width="0.1524" layer="91"/>
-<label x="0" y="-109.22" size="1.778" layer="95"/>
+<pinref part="TP3" gate="G$1" pin="TP"/>
+<wire x1="-5.08" y1="-124.46" x2="0" y2="-124.46" width="0.1524" layer="91"/>
+<label x="0" y="-124.46" size="1.778" layer="95"/>
 </segment>
 </net>
@@
 </segment>
 <segment>
-<pinref part="TP3" gate="G$1" pin="TP"/>
+<pinref part="MISO" gate="G$1" pin="TP"/>
 <wire x1="-5.08" y1="-88.9" x2="0" y2="-88.9" width="0.1524" layer="91"/>
 <label x="0" y="-88.9" size="1.778" layer="95"/>
@@
 </segment>
 <segment>
-<pinref part="TP2" gate="G$1" pin="TP"/>
+<pinref part="MOSI" gate="G$1" pin="TP"/>
 <wire x1="-5.08" y1="-78.74" x2="0" y2="-78.74" width="0.1524" layer="91"/>
 <label x="0" y="-78.74" size="1.778" layer="95"/>
