File: device/POC/BikeLight POC.sch (EAGLE design)
At the start: 43 parts, among them IC1 MCP2515-I-ML, IC10 MCP1802T-5002I/OT, IC2 MICROSD_SPI_MODE, IC3 FM25W256-SOIC, IC4 MCP2561-2, IC5 TXB0106, IC6 PRQV8.00CR1510Y00L, IC7 ADXL345, IC8 74HCT1G32, IC9 MCP1802T-3302I/OT

Commit message: - decided to power the power indicator LED from 5V0 instead from the battery directly
Connections:
- net !SNDN!: no longer LED1.A
- net 5V0: now also LED1.A
Other:
- note added: "SPI Test Pads"
- moved on the sheet: CAN_GND, LED1, MISO, MOSI, R9, SCK, TP1, TP2, TP3, TP4
Changed lines of the file:
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@@
 <text x="274.32" y="58.42" size="1.778" layer="90">CAN Bus Transciever</text>
 <text x="165.1" y="60.96" size="1.778" layer="90">CAN Bus Controller</text>
+<text x="-15.24" y="-101.6" size="1.778" layer="90">SPI Test Pads</text>
 </plain>
 <instances>
@@
 <instance part="R8" gate="G$1" x="101.6" y="-175.26" rot="R90"/>
 <instance part="IC8" gate="G$1" x="365.76" y="-48.26" rot="R180"/>
-<instance part="CAN_GND" gate="G$1" x="-7.62" y="-68.58" rot="R270"/>
-<instance part="MOSI" gate="G$1" x="-7.62" y="-78.74" rot="R270"/>
-<instance part="MISO" gate="G$1" x="-7.62" y="-88.9" rot="R270"/>
-<instance part="SCK" gate="G$1" x="-7.62" y="-99.06" rot="R270"/>
-<instance part="TP3" gate="G$1" x="-7.62" y="-124.46" rot="R90"/>
-<instance part="TP2" gate="G$1" x="-7.62" y="-116.84" rot="R90"/>
-<instance part="TP4" gate="G$1" x="-7.62" y="-132.08" rot="R90"/>
-<instance part="TP1" gate="G$1" x="-7.62" y="-109.22" rot="R90"/>
-<instance part="LED1" gate="G$1" x="101.6" y="-165.1" rot="R180"/>
-<instance part="R9" gate="G$1" x="101.6" y="-154.94" rot="R90"/>
+<instance part="CAN_GND" gate="G$1" x="393.7" y="20.32" rot="R90"/>
+<instance part="MOSI" gate="G$1" x="-7.62" y="-111.76" rot="R270"/>
+<instance part="MISO" gate="G$1" x="-7.62" y="-121.92" rot="R270"/>
+<instance part="SCK" gate="G$1" x="-7.62" y="-132.08" rot="R270"/>
+<instance part="TP3" gate="G$1" x="-7.62" y="-157.48" rot="R90"/>
+<instance part="TP2" gate="G$1" x="-7.62" y="-149.86" rot="R90"/>
+<instance part="TP4" gate="G$1" x="-7.62" y="-165.1" rot="R90"/>
+<instance part="TP1" gate="G$1" x="-7.62" y="-142.24" rot="R90"/>
+<instance part="LED1" gate="G$1" x="109.22" y="-154.94" rot="R90"/>
+<instance part="R9" gate="G$1" x="119.38" y="-154.94"/>
 </instances>
 <busses>
@@
 <segment>
 <pinref part="CAN_GND" gate="G$1" pin="TP"/>
-<wire x1="-5.08" y1="-68.58" x2="0" y2="-68.58" width="0.1524" layer="91"/>
-<label x="0" y="-68.58" size="1.778" layer="95"/>
+<wire x1="391.16" y1="20.32" x2="381" y2="20.32" width="0.1524" layer="91"/>
+<label x="381" y="20.32" size="1.778" layer="95"/>
 </segment>
 <segment>
 <pinref part="R9" gate="G$1" pin="2"/>
-<wire x1="101.6" y1="-149.86" x2="101.6" y2="-147.32" width="0.1524" layer="91"/>
-<label x="101.6" y="-147.32" size="1.778" layer="95"/>
+<wire x1="124.46" y1="-154.94" x2="127" y2="-154.94" width="0.1524" layer="91"/>
+<label x="127" y="-154.94" size="1.778" layer="95" rot="R270"/>
 </segment>
 </net>
@@
 <pinref part="IC8" gate="G$1" pin="VCC"/>
 </segment>
+<segment>
+<pinref part="LED1" gate="G$1" pin="A"/>
+<wire x1="106.68" y1="-154.94" x2="99.06" y2="-154.94" width="0.1524" layer="91"/>
+<label x="99.06" y="-154.94" size="1.778" layer="95"/>
+</segment>
 </net>
 <net name="OSC1" class="0">
@@
 <segment>
 <pinref part="TP2" gate="G$1" pin="TP"/>
-<wire x1="-5.08" y1="-116.84" x2="0" y2="-116.84" width="0.1524" layer="91"/>
-<label x="0" y="-116.84" size="1.778" layer="95"/>
+<wire x1="-5.08" y1="-149.86" x2="0" y2="-149.86" width="0.1524" layer="91"/>
+<label x="0" y="-149.86" size="1.778" layer="95"/>
 </segment>
 </net>
@@
 <wire x1="101.6" y1="-170.18" x2="109.22" y2="-170.18" width="0.1524" layer="91"/>
 <junction x="101.6" y="-170.18"/>
-<pinref part="LED1" gate="G$1" pin="A"/>
-<wire x1="101.6" y1="-170.18" x2="101.6" y2="-167.64" width="0.1524" layer="91"/>
 </segment>
 </net>
@@
 <segment>
 <pinref part="TP4" gate="G$1" pin="TP"/>
-<wire x1="-5.08" y1="-132.08" x2="0" y2="-132.08" width="0.1524" layer="91"/>
-<label x="0" y="-132.08" size="1.778" layer="95"/>
+<wire x1="-5.08" y1="-165.1" x2="0" y2="-165.1" width="0.1524" layer="91"/>
+<label x="0" y="-165.1" size="1.778" layer="95"/>
 </segment>
 </net>
@@
 <segment>
 <pinref part="SCK" gate="G$1" pin="TP"/>
-<wire x1="-5.08" y1="-99.06" x2="0" y2="-99.06" width="0.1524" layer="91"/>
-<label x="0" y="-99.06" size="1.778" layer="95"/>
+<wire x1="-5.08" y1="-132.08" x2="0" y2="-132.08" width="0.1524" layer="91"/>
+<label x="0" y="-132.08" size="1.778" layer="95"/>
 </segment>
 </net>
@@
 <segment>
 <pinref part="TP1" gate="G$1" pin="TP"/>
-<wire x1="-5.08" y1="-109.22" x2="0" y2="-109.22" width="0.1524" layer="91"/>
-<label x="0" y="-109.22" size="1.778" layer="95"/>
+<wire x1="-5.08" y1="-142.24" x2="0" y2="-142.24" width="0.1524" layer="91"/>
+<label x="0" y="-142.24" size="1.778" layer="95"/>
 </segment>
 </net>
@@
 <segment>
 <pinref part="TP3" gate="G$1" pin="TP"/>
-<wire x1="-5.08" y1="-124.46" x2="0" y2="-124.46" width="0.1524" layer="91"/>
-<label x="0" y="-124.46" size="1.778" layer="95"/>
+<wire x1="-5.08" y1="-157.48" x2="0" y2="-157.48" width="0.1524" layer="91"/>
+<label x="0" y="-157.48" size="1.778" layer="95"/>
 </segment>
 </net>
@@
 <segment>
 <pinref part="MISO" gate="G$1" pin="TP"/>
-<wire x1="-5.08" y1="-88.9" x2="0" y2="-88.9" width="0.1524" layer="91"/>
-<label x="0" y="-88.9" size="1.778" layer="95"/>
+<wire x1="-5.08" y1="-121.92" x2="0" y2="-121.92" width="0.1524" layer="91"/>
+<label x="0" y="-121.92" size="1.778" layer="95"/>
 </segment>
 </net>
@@
 <segment>
 <pinref part="MOSI" gate="G$1" pin="TP"/>
-<wire x1="-5.08" y1="-78.74" x2="0" y2="-78.74" width="0.1524" layer="91"/>
-<label x="0" y="-78.74" size="1.778" layer="95"/>
-</segment>
-</net>
+<wire x1="-5.08" y1="-111.76" x2="0" y2="-111.76" width="0.1524" layer="91"/>
+<label x="0" y="-111.76" size="1.778" layer="95"/>
+</segment>
+</net>
